Commit message: Cart and PSM models, controllers not working

File: dvrk_model/urdf/ECM.urdf (robot description, URDF)
Before this commit: robot ecm, 8 links, 7 joints
Links:
- added link ecm_base_link, mass 0.01; collision mesh filename=package://dvrk_model/meshes/ecm/ECM_Base.STL scale=0.001 0.001 0.001; visual mesh filename=package://dvrk_model/meshes/ecm/ECM_Base.STL scale=0.001 0.001 0.001
- link ecm_pitch_link: mass None -> 0.01
Joints:
- added joint fixed_joint: type fixed, parent world, child ecm_base_link, origin xyz=0 0.0 0.0 rpy=0.0 0.0 0.0
- joint outer_yaw: origin xyz=-0.6 0.1 0 rpy=-1.570795 0 -1.570795 -> xyz=-0.76 -0.075 -0.0775 rpy=-1.570795 0 -1.570795; parent world -> ecm_base_link

File: dvrk_model/urdf/dvrk.urdf.xacro (robot description, xacro)
@@ -14,5 +14,5 @@
       prefix="one_"
       parent_link="world"
-      xyz= "0 0 0" rpy="0.0 0.0 3.1415926"
+      xyz= "0 0 0" rpy="0.0 0.0 0"
      />
       <!-- "-0.5 0.0 1"    -->

File: dvrk_model/urdf/dvrk_t1_1.xacro (robot description, xacro)
@@ -9,8 +9,8 @@
       xyz="0.5 0.0 1.0" rpy="0.0 0.0 0.0"/>-->
   <!-- Macros -->
- <xacro:include filename="$(find dvrk_model)/Cart/urdf/Cart_n.xacro"/>
- <xacro:include filename="$(find dvrk_model)/urdf/psm.xacro"/>
- <!--<xacro:include filename="$(find dvrk_model)/urdf/psm_parallel.urdf.xacro"/>-->
- <xacro:include filename="$(find dvrk_model)/urdf/ecm.urdf.xacro"/>
+ <xacro:include filename="$(find dvrk_model)/Cart/Cart_n.xacro"/>
+ <!-- <xacro:include filename="$(find dvrk_model)/urdf/psm.xacro"/> -->
+ <!-- <xacro:include filename="$(find dvrk_model)/PSM/psm_parallel.urdf.xacro"/>
+ <xacro:include filename="$(find dvrk_model)/ECM/ecm.urdf.xacro"/> -->
 <!--specify how many psms:(1 to 3) change true to one of the values-->
 <property name= "psm_num_1" value = "true" />
@@ -22,7 +22,9 @@
 <property name= "psm3" value= "4" />
 <property name="if" value="1" />
+<xacro:Cart prefix="Cart/"/>
  <xacro:if value="${psm_num_1}">
-   	<xacro:psm prefix="1" parent="${psm1}"  />
-	<xacro:ecm prefix="ecm" parent_link="C_A2_L3" xyz="0.0 0.0 0.0" rpy="0.0 0.0 0.0"  />
+  <!-- <xacro:psm prefix="PSM1::one_" parent_link="C_A1_L4" xyz= "0 0 0" rpy="0 0 0"/> -->
+   	<!-- <xacro:psm prefix="one_" parent="${psm1}"  /> -->
+	<!-- <xacro:ecm prefix="ecm" parent_link="C_A2_L3" xyz="0.16 0.125 0.075" rpy="0.0 0 -${3.14159/4-0.05}"  /> -->
  </xacro:if>
  <xacro:if value="${psm_num_2}">
@@ -31,8 +33,11 @@
  </xacro:if>
  <xacro:if value="${psm_num_3}">
-   	<xacro:psm prefix="1" parent="1"  />
+   	<!-- <xacro:psm prefix="1" parent="1"  />
 	<xacro:psm prefix="2" parent="3"  />
-	<xacro:psm prefix="3" parent="4"  />
-	<xacro:ecm prefix="ecm" parent_link="C_A2_L3" xyz="0.0 0.0 0.0" rpy="0.0 0.0 0.0"  />
+	<xacro:psm prefix="3" parent="4"  /> -->
+  <xacro:psm prefix="PSM1::one_" parent_link="C_A1_L4" xyz= "0 0 0" rpy="0 0 0"/>
+  <xacro:psm prefix="PSM2::one_" parent_link="C_A3_L4" xyz= "0 0 0" rpy="0 0 0"/>
+  <xacro:psm prefix="PSM3::one_" parent_link="C_A4_L4" xyz= "0 0 0" rpy="0 0 0"/>
+	<xacro:ecm prefix="ecm" parent_link="C_A2_L3" xyz="0.16 0.125 0.075" rpy="0.0 0 -${3.14159/4-0.05}"  />
  </xacro:if>
       <!-- "-0.5 0.0 1"    -->
@@ -41,8 +46,8 @@
       parent_link="world"
       xyz="-0.5 -0.1 0.82949" rpy="0 -1.570796 0.0"/> -->
-  <gazebo>
+  <!-- <gazebo>
   <plugin name="gazebo_ros_control" filename="libgazebo_ros_control.so">
   <robotSimType>gazebo_ros_control/DefaultRobotHWSim</robotSimType>
   </plugin>
-  </gazebo>
+  </gazebo> -->
 </robot>

File: dvrk_model/urdf/ecm.urdf.xacro (robot description, xacro)
@@ -35,16 +35,36 @@
     </link>-->
     <!-- Joint 0: Fixed to Setup Joint-->
-    <!--<joint name="fixed_joint" type="fixed">
+    <joint name="fixed_joint" type="fixed">
       <parent link="${parent_link}"/>
       <child link="${prefix}_base_link"/>
-      <origin rpy="0 0 0" xyz="0.38866 0 -0.46107"/>
-    </joint>
-    <link name="${prefix}_base_link"/>-->
+      <origin rpy="${rpy}" xyz="${xyz}"/>
+    </joint>
+    <link name="${prefix}_base_link">
+      <inertial>
+        <mass value="0.01"/>
+        <origin rpy="0 0 0" xyz="0.0 0 0"/>
+        <inertia ixx="1.0" ixy="0.0" ixz="0.0" iyy="1.0" iyz="0.0" izz="1.0"/>
+      </inertial>
+      <visual>
+        <origin rpy="0 ${3.14159/2} ${3.14159}" xyz="0.0 0 0"/>
+        <geometry>
+          <mesh filename="package://dvrk_model/meshes/ecm/ECM_Base.STL" scale="0.001 0.001 0.001"/>
+        </geometry>
+	<material name="DaVinciGreen"/>
+      </visual>
+      <collision>
+        <origin rpy="0 ${3.14159/2} ${3.14159}" xyz="0.0 0 0"/>
+        <geometry>
+          <mesh filename="package://dvrk_model/meshes/ecm/ECM_Base.STL" scale="0.001 0.001 0.001"/>
+        </geometry>
+      </collision>
+    </link>
     <!-- Joint 1: Outer Yaw -->
     <joint name="outer_yaw" type="revolute">
-      <parent link="${parent_link}"/>
+      <parent link="${prefix}_base_link"/>
       <child link="${prefix}_yaw_link"/>
       <!--<origin rpy="0 -${3.14159/2} ${3.14159/2}" xyz="0 0 0"/>-->
-      <origin rpy="-${3.14159/2} 0 -${3.14159/2}" xyz="-0.6 0.1 0"/>
+      <!--<origin rpy="-${3.14159/2} 0 -${3.14159/2}" xyz="-0.6 0.1 0"/>-->
+      <origin rpy="-${3.14159/2} 0 -${3.14159/2}" xyz="-0.76 -0.075 -0.0775"/>
       <axis xyz="0 0 1"/>
       <!--rotates about z axis-->
