Commit message: Tested on hardware, everything works

File: dvrk_model/urdf/LaprotekMaster.urdf (robot description, URDF)
Before this commit: robot LaprotekMaster, 16 links, 15 joints
Joints:
- joint right_forarm_axis: axis 1 0 0 -> -1 0 0
