Commit message: Laprotek urdf updated

File: dvrk_model/LaprotekMaster/LaprotekMaster.urdf (robot description, URDF)
Before this commit: robot LaprotekMaster, 16 links, 15 joints
Links:
- removed link left_forarm_link
- removed link left_grip_link
- removed link left_inner_link
- removed link left_outer_joint
- removed link left_shoulder_link
- removed link left_thumb_link
- removed link left_twist_joint
Joints:
- removed joint left_forarm_axis
- removed joint left_grip_axis
- removed joint left_inner_axis
- removed joint left_outer_axis
- removed joint left_shoulder_axis
- removed joint left_thumb_axis
- removed joint left_twist_axis
- joint right_grip_axis: axis -0.642787609686614 0 0.766044443118915 -> 0 0 1
- joint right_inner_axis: axis 0 0 0 -> 0 0 1; type fixed -> revolute
- joint right_outer_axis: axis -1 0 0 -> 1 0 0
