Commit message: modified ros control plugin

File: dvrk_model/ECM/ecm.urdf.xacro (robot description, xacro)
@@ -1,4 +1,15 @@
 <?xml version="1.0" ?>
 <robot name="ecm" xmlns:xacro="http://www.ros.org/wiki/xacro">
+  <xacro:macro name="transmission_tags" params = "joint_name mech_red hw_intf">
+    <transmission name="${joint_name}_trans">
+      <type>transmission_interface/SimpleTransmission</type>
+      <joint name="${joint_name}">
+        <hardwareInterface> ${hw_intf} </hardwareInterface>
+      </joint>
+      <actuator name="${joint_name}_motor">
+        <mechanicalReduction>${mech_red}</mechanicalReduction>
+      </actuator>
+    </transmission>
+  </xacro:macro>
   <!-- Macro for da Vinci Endoscope Camera Manipulator (ECM) -->
   <xacro:macro name="ecm" params="prefix parent_link xyz rpy">
@@ -7,9 +18,9 @@
     <joint name="fixed_joint" type="fixed">
       <parent link="${parent_link}"/>
-      <child link="${prefix}_base_link"/>
+      <child link="${prefix}base_link"/>
       <origin rpy="${rpy}" xyz="${xyz}"/>
     </joint>
     <link
-      name="${prefix}_base_link">
+      name="${prefix}base_link">
       <inertial>
         <origin
@@ -51,5 +62,5 @@
     </link>
     <link
-      name="${prefix}_yaw_link">
+      name="${prefix}yaw_link">
       <inertial>
         <origin
@@ -91,5 +102,5 @@
     </link>
     <joint
-      name="${prefix}_yaw_joint"
+      name="${prefix}yaw_joint"
       type="revolute">
       <origin
@@ -97,7 +108,7 @@
         rpy="1.57079632679615 -3.58046925441613E-13 1.5707963267949" />
       <parent
-        link="${prefix}_base_link" />
-      <child
-        link="${prefix}_yaw_link" />
+        link="${prefix}base_link" />
+      <child
+        link="${prefix}yaw_link" />
       <axis
         xyz="0 0 1" />
@@ -109,5 +120,5 @@
     </joint>
     <link
-      name="${prefix}_pitch_front_link">
+      name="${prefix}pitch_front_link">
       <inertial>
         <origin
@@ -149,5 +160,5 @@
     </link>
     <joint
-      name="${prefix}_pitch_front_joint"
+      name="${prefix}pitch_front_joint"
       type="revolute">
       <origin
@@ -155,7 +166,7 @@
         rpy="3.14 -1.5707963267949 0" />
       <parent
-        link="${prefix}_yaw_link" />
-      <child
-        link="${prefix}_pitch_front_link" />
+        link="${prefix}yaw_link" />
+      <child
+        link="${prefix}pitch_front_link" />
       <axis
         xyz="0 0 1" />
@@ -167,5 +178,5 @@
     </joint>
     <link
-      name="${prefix}_pitch_bottom_link">
+      name="${prefix}pitch_bottom_link">
       <inertial>
         <origin
@@ -207,5 +218,5 @@
     </link>
     <joint
-      name="${prefix}_pitch_bottom_joint"
+      name="${prefix}pitch_bottom_joint"
       type="revolute">
       <origin
@@ -213,7 +224,7 @@
         rpy="0 0 0" />
       <parent
-        link="${prefix}_pitch_front_link" />
-      <child
-        link="${prefix}_pitch_bottom_link" />
+        link="${prefix}pitch_front_link" />
+      <child
+        link="${prefix}pitch_bottom_link" />
       <axis
         xyz="0 0 1" />
@@ -223,8 +234,8 @@
         effort="1000"
         velocity="10" />
-      <mimic joint="${prefix}_pitch_front_joint" multiplier="-1"/>
-    </joint>
-    <link
-      name="${prefix}_pitch_end_link">
+      <mimic joint="${prefix}pitch_front_joint" multiplier="-1"/>
+    </joint>
+    <link
+      name="${prefix}pitch_end_link">
       <inertial>
         <origin
@@ -266,5 +277,5 @@
     </link>
     <joint
-      name="${prefix}_pitch_end_joint"
+      name="${prefix}pitch_end_joint"
       type="revolute">
       <origin
@@ -272,7 +283,7 @@
         rpy="0 0 0" />
       <parent
-        link="${prefix}_pitch_bottom_link" />
-      <child
-        link="${prefix}_pitch_end_link" />
+        link="${prefix}pitch_bottom_link" />
+      <child
+        link="${prefix}pitch_end_link" />
       <axis
         xyz="0 0 1" />
@@ -282,8 +293,8 @@
         effort="1000"
         velocity="10" />
-      <mimic joint="${prefix}_pitch_front_joint" multiplier="1"/>
-    </joint>
-    <link
-      name="${prefix}_main_insertion_link">
+      <mimic joint="${prefix}pitch_front_joint" multiplier="1"/>
+    </joint>
+    <link
+      name="${prefix}main_insertion_link">
       <inertial>
         <origin
@@ -325,5 +336,5 @@
     </link>
     <joint
-      name="${prefix}_main_insertion_joint"
+      name="${prefix}main_insertion_joint"
       type="prismatic">
       <origin
@@ -331,7 +342,7 @@
         rpy="-1.5708 0 0" />
       <parent
-        link="${prefix}_pitch_end_link" />
-      <child
-        link="${prefix}_main_insertion_link" />
+        link="${prefix}pitch_end_link" />
+      <child
+        link="${prefix}main_insertion_link" />
       <axis
         xyz="0 0 1" />
@@ -343,5 +354,5 @@
     </joint>
     <link
-      name="${prefix}_tool_link">
+      name="${prefix}tool_link">
       <inertial>
         <origin
@@ -383,5 +394,5 @@
     </link>
     <joint
-      name="${prefix}_tool_joint"
+      name="${prefix}tool_joint"
       type="revolute">
       <origin
@@ -389,7 +400,7 @@
         rpy="0 0 0" />
       <parent
-        link="${prefix}_main_insertion_link" />
-      <child
-        link="${prefix}_tool_link" />
+        link="${prefix}main_insertion_link" />
+      <child
+        link="${prefix}tool_link" />
       <axis
         xyz="0 0 -1" />
@@ -401,5 +412,5 @@
     </joint>
     <link
-      name="${prefix}_pitch_top_link">
+      name="${prefix}pitch_top_link">
       <inertial>
         <origin
@@ -441,5 +452,5 @@
     </link>
     <joint
-      name="${prefix}_pitch_top_joint"
+      name="${prefix}pitch_top_joint"
       type="revolute">
       <origin
@@ -447,7 +458,7 @@
         rpy="0 0 0" />
       <parent
-        link="${prefix}_pitch_front_link" />
-      <child
-        link="${prefix}_pitch_top_link" />
+        link="${prefix}pitch_front_link" />
+      <child
+        link="${prefix}pitch_top_link" />
       <axis
         xyz="0 0 1" />
@@ -457,8 +468,8 @@
         effort="1000"
         velocity="10" />
-      <mimic joint="${prefix}_pitch_front_joint" multiplier="-1"/>
-    </joint>
-    <link
-      name="${prefix}_pitch_back_link">
+      <mimic joint="${prefix}pitch_front_joint" multiplier="-1"/>
+    </joint>
+    <link
+      name="${prefix}pitch_back_link">
       <inertial>
         <origin
@@ -500,5 +511,5 @@
     </link>
     <joint
-      name="${prefix}_pitch_back_joint"
+      name="${prefix}pitch_back_joint"
       type="revolute">
       <origin
@@ -506,7 +517,7 @@
         rpy="3.14 -1.5707963267949 0" />
       <parent
-        link="${prefix}_yaw_link" />
-      <child
-        link="${prefix}_pitch_back_link" />
+        link="${prefix}yaw_link" />
+      <child
+        link="${prefix}pitch_back_link" />
       <axis
         xyz="0 0 1" />
@@ -516,8 +527,8 @@
         effort="1000"
         velocity="10" />
-      <mimic joint="${prefix}_pitch_front_joint" multiplier="1"/>
-    </joint>
-    <link
-      name="${prefix}_remote_center_link">
+      <mimic joint="${prefix}pitch_front_joint" multiplier="1"/>
+    </joint>
+    <link
+      name="${prefix}remote_center_link">
       <inertial>
         <origin
@@ -559,5 +570,5 @@
     </link>
     <joint
-      name="${prefix}_remote_center_joint"
+      name="${prefix}remote_center_joint"
       type="fixed">
       <origin
@@ -565,13 +576,13 @@
         rpy="-1.249734375614E-12 3.58046925441613E-13 -1.5707963267949" />
       <parent
-        link="${prefix}_base_link" />
-      <child
-        link="${prefix}_remote_center_link" />
+        link="${prefix}base_link" />
+      <child
+        link="${prefix}remote_center_link" />
       <axis
         xyz="0 0 0" />
     </joint>
-    <link name="${prefix}_end_link"/>
-    <joint
-      name="${prefix}_end_joint"
+    <link name="${prefix}end_link"/>
+    <joint
+      name="${prefix}end_joint"
       type="fixed">
       <origin
@@ -579,10 +590,14 @@
         rpy="0 0 0" />
       <parent
-        link="${prefix}_tool_link" />
-      <child
-        link="${prefix}_end_link" />
+        link="${prefix}tool_link" />
+      <child
+        link="${prefix}end_link" />
       <axis
         xyz="0 0 0" />
     </joint>
+  <xacro:transmission_tags joint_name="${prefix}yaw_joint" mech_red = "1" hw_intf= "hardware_interface/EffortJointInterface" />
+  <xacro:transmission_tags joint_name="${prefix}pitch_front_joint" mech_red = "1" hw_intf= "hardware_interface/EffortJointInterface" />
+  <xacro:transmission_tags joint_name="${prefix}main_insertion_joint" mech_red = "1" hw_intf= "hardware_interface/EffortJointInterface" />
+  <xacro:transmission_tags joint_name="${prefix}tool_joint" mech_red = "1" hw_intf= "hardware_interface/EffortJointInterface" />
   </xacro:macro>
 </robot>

File: dvrk_model/PSM/psm.urdf.xacro (robot description, xacro)
@@ -1,4 +1,15 @@
 <?xml version="1.0" encoding="utf-8"?>
 <robot name="PSM" xmlns:xacro="http://www.ros.org/wiki/xacro">
+  <xacro:macro name="transmission_tags" params = "joint_name mech_red hw_intf">
+    <transmission name="${joint_name}_trans">
+      <type>transmission_interface/SimpleTransmission</type>
+      <joint name="${joint_name}">
+        <hardwareInterface> ${hw_intf} </hardwareInterface>
+      </joint>
+      <actuator name="${joint_name}_motor">
+        <mechanicalReduction>${mech_red}</mechanicalReduction>
+      </actuator>
+    </transmission>
+  </xacro:macro>
   <xacro:macro name="psm" params=" prefix parent_link xyz rpy">
     <joint name="${prefix}rev_joint" type="revolute">
@@ -469,4 +480,7 @@
     <origin rpy="0 0 -1.5708" xyz="0.4864 0 0.1524"/>
   </joint>
+  <xacro:transmission_tags joint_name="${prefix}yaw_joint" mech_red = "1" hw_intf= "hardware_interface/EffortJointInterface" />
+  <xacro:transmission_tags joint_name="${prefix}pitch_back_joint" mech_red = "1" hw_intf= "hardware_interface/EffortJointInterface" />
+  <xacro:transmission_tags joint_name="${prefix}main_insertion_joint" mech_red = "1" hw_intf= "hardware_interface/EffortJointInterface" />
   </xacro:macro>
 </robot>

File: dvrk_model/Tool_LND/tool_lnd.urdf.xacro (robot description, xacro)
@@ -2,4 +2,15 @@
 <robot name="LargeNeedleDriver" xmlns:xacro="http://www.ros.org/wiki/xacro">
   <xacro:macro name="tool_lnd" params=" prefix parent_link xyz rpy">
+  <xacro:macro name="transmission_tags" params = "joint_name mech_red hw_intf">
+    <transmission name="${joint_name}_trans">
+      <type>transmission_interface/SimpleTransmission</type>
+      <joint name="${joint_name}">
+        <hardwareInterface> ${hw_intf} </hardwareInterface>
+      </joint>
+      <actuator name="${joint_name}_motor">
+        <mechanicalReduction>${mech_red}</mechanicalReduction>
+      </actuator>
+    </transmission>
+  </xacro:macro>
   <joint name="${prefix}tool_joint" type="fixed">
    <parent link="${parent_link}"/>
@@ -344,4 +355,9 @@
     <origin rpy="3.14159265358979 0 -0.28511888006" xyz="0 0 0"/>
   </joint>
+  <xacro:transmission_tags joint_name="${prefix}tool_roll_joint" mech_red = "1" hw_intf= "hardware_interface/EffortJointInterface" />
+  <xacro:transmission_tags joint_name="${prefix}tool_pitch_joint" mech_red = "1" hw_intf= "hardware_interface/EffortJointInterface" />
+  <xacro:transmission_tags joint_name="${prefix}tool_yaw_joint" mech_red = "1" hw_intf= "hardware_interface/EffortJointInterface" />
+  <xacro:transmission_tags joint_name="${prefix}gripper1_joint" mech_red = "1" hw_intf= "hardware_interface/EffortJointInterface" />
+  <xacro:transmission_tags joint_name="${prefix}gripper2_joint" mech_red = "1" hw_intf= "hardware_interface/EffortJointInterface" />
   </xacro:macro>
 </robot>
